File: electronics/kicad/actuator_y.kicad_sch (KiCad schematic)
At the start: 14 parts, among them U17 DRV8212PDSG, U18 INA241A1, U19 LMV331, U20 LMV331

Commit message: Firmware review follow-up: ICD v1.3, parameters v0.4.3, thermal and headroom corrections
Resolves on the upstream side the discrepancies D1-D12 found by the
firmware workstream:
- ICD v1.3 (docs/icd.md). D1: the Jacobian was printed inverted; it is
  Rot(phi) diag(J_t1, 1) Rot(rho). D2: the actuator force sign is
  -n Kf i at the tip. D7: gamma is tilt-dependent, so CAL_USER v2 stores
  r_n = K_n/k_ax. D8: optics run at 1 kHz. D4: the calibration
  container and the 0x04/0x05 payloads are defined, and the mode codes
  added. The page origin, 64-bit stroke time and boundary samples are
  documented as implemented. ML contract v1.2 adds confidence rule (5)
  and the status of the exported artefact.
- D6 and thermal model: analysis/thermal.py read a 0.45 mm air gap and
  60 mW of electronics. At 0.50 mm and 115 mW it gives coil-to-structure
  145 K/W, 157 K/W steady to ambient, allowable 0.412 W (was 0.455;
  now set by the 120 C coil limit) and a Rev A coil of 96.6 C. It also
  emits a two-node governor model.
- config v0.4.3: actuator.air_gap, Rth_coil_amb 145 K/W, and structure
  node parameters.
- D11: electronics/calcs/drive_sense.py headroom now uses per-point
  coil and magnet temperatures, the Br tempco and the correction force.
  At 3.3 V the 6 ohm winding cannot hold 0.5 % of the thermal envelope;
  4 ohm can. 6 ohm stays the baseline (DEC-012 revisited, EXP-B03 winds
  both). The baseline winding, not the assessment, now drives the
  ripple, loop and hold current.
- D3: the H-bridge note is corrected (slow decay = one input high).
  Schematic UUIDs are now deterministic; ERC shows 0 errors and 1
  accepted warning; the netlist check passes (102 nets, 492 pins).
- sim/pensim/model.py reads its bandwidths from the YAML (values
  unchanged; 12 tests pass). D9 and D10 are recorded as simulator
  limitations.
- Docs, requirements (REQ-ACT-001, REQ-THM-002; REQ-CTRL-002 at risk at
  a 35.3 deg phase margin), validation predictions and criteria
  (AC-B03-08 now mea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
Other:
- note added: "IN/IN drive (DRV8212P truth table, VERIFY): slow decay = one input held high, the other driven with the inverted duty, i.e. drive (1,0) / brake (1,1). PWM on one input with the other low is drive/coast (fast decay). nSLEEP low = sleep, outputs Hi-Z. Centre-aligned PWM, current sampled at period centre."
- note removed: "IN/IN drive: PWM on one input, other low = drive/brake (slow decay); both low + SLEEP low = coast. Centre-aligned PWM, current sampled at period centre."
Changed lines of the file:
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@@
     (instances
       (project "pen_research"
-        (path "/8dc8c6c6-b52c-4ea1-b54e-983058d7675b/f0a18f19-96a9-433d-b9f0-5a690030b810"
+        (path "/f9a5e985-59a4-50af-9b9a-f23ea55006e2/ddb8b498-860e-5487-980d-a3b64ae1ae94"
           (reference "U17")
           (unit 1)))))
@@
     (instances
       (project "pen_research"
-        (path "/8dc8c6c6-b52c-4ea1-b54e-983058d7675b/f0a18f19-96a9-433d-b9f0-5a690030b810"
+        (path "/f9a5e985-59a4-50af-9b9a-f23ea55006e2/ddb8b498-860e-5487-980d-a3b64ae1ae94"
           (reference "C60")
           (unit 1)))))
@@
     (instances
       (project "pen_research"
-        (path "/8dc8c6c6-b52c-4ea1-b54e-983058d7675b/f0a18f19-96a9-433d-b9f0-5a690030b810"
+        (path "/f9a5e985-59a4-50af-9b9a-f23ea55006e2/ddb8b498-860e-5487-980d-a3b64ae1ae94"
           (reference "C61")
           (unit 1)))))
@@
     (instances
       (project "pen_research"
-        (path "/8dc8c6c6-b52c-4ea1-b54e-983058d7675b/f0a18f19-96a9-433d-b9f0-5a690030b810"
+        (path "/f9a5e985-59a4-50af-9b9a-f23ea55006e2/ddb8b498-860e-5487-980d-a3b64ae1ae94"
           (reference "C62")
           (unit 1)))))
@@
     (instances
       (project "pen_research"
-        (path "/8dc8c6c6-b52c-4ea1-b54e-983058d7675b/f0a18f19-96a9-433d-b9f0-5a690030b810"
+        (path "/f9a5e985-59a4-50af-9b9a-f23ea55006e2/ddb8b498-860e-5487-980d-a3b64ae1ae94"
           (reference "R50")
           (unit 1)))))
@@
     (instances
       (project "pen_research"
-        (path "/8dc8c6c6-b52c-4ea1-b54e-983058d7675b/f0a18f19-96a9-433d-b9f0-5a690030b810"
+        (path "/f9a5e985-59a4-50af-9b9a-f23ea55006e2/ddb8b498-860e-5487-980d-a3b64ae1ae94"
           (reference "U18")
           (unit 1)))))
@@
     (instances
       (project "pen_research"
-        (path "/8dc8c6c6-b52c-4ea1-b54e-983058d7675b/f0a18f19-96a9-433d-b9f0-5a690030b810"
+        (path "/f9a5e985-59a4-50af-9b9a-f23ea55006e2/ddb8b498-860e-5487-980d-a3b64ae1ae94"
           (reference "C63")
           (unit 1)))))
@@
     (instances
       (project "pen_research"
-        (path "/8dc8c6c6-b52c-4ea1-b54e-983058d7675b/f0a18f19-96a9-433d-b9f0-5a690030b810"
+        (path "/f9a5e985-59a4-50af-9b9a-f23ea55006e2/ddb8b498-860e-5487-980d-a3b64ae1ae94"
           (reference "R51")
           (unit 1)))))
@@
     (instances
       (project "pen_research"
-        (path "/8dc8c6c6-b52c-4ea1-b54e-983058d7675b/f0a18f19-96a9-433d-b9f0-5a690030b810"
+        (path "/f9a5e985-59a4-50af-9b9a-f23ea55006e2/ddb8b498-860e-5487-980d-a3b64ae1ae94"
           (reference "C64")
           (unit 1)))))
@@
     (instances
       (project "pen_research"
-        (path "/8dc8c6c6-b52c-4ea1-b54e-983058d7675b/f0a18f19-96a9-433d-b9f0-5a690030b810"
+        (path "/f9a5e985-59a4-50af-9b9a-f23ea55006e2/ddb8b498-860e-5487-980d-a3b64ae1ae94"
           (reference "TP26")
           (unit 1)))))
@@
     (instances
       (project "pen_research"
-        (path "/8dc8c6c6-b52c-4ea1-b54e-983058d7675b/f0a18f19-96a9-433d-b9f0-5a690030b810"
+        (path "/f9a5e985-59a4-50af-9b9a-f23ea55006e2/ddb8b498-860e-5487-980d-a3b64ae1ae94"
           (reference "TP27")
           (unit 1)))))
@@
     (instances
       (project "pen_research"
-        (path "/8dc8c6c6-b52c-4ea1-b54e-983058d7675b/f0a18f19-96a9-433d-b9f0-5a690030b810"
+        (path "/f9a5e985-59a4-50af-9b9a-f23ea55006e2/ddb8b498-860e-5487-980d-a3b64ae1ae94"
           (reference "U19")
           (unit 1)))))
@@
     (instances
       (project "pen_research"
-        (path "/8dc8c6c6-b52c-4ea1-b54e-983058d7675b/f0a18f19-96a9-433d-b9f0-5a690030b810"
+        (path "/f9a5e985-59a4-50af-9b9a-f23ea55006e2/ddb8b498-860e-5487-980d-a3b64ae1ae94"
           (reference "U20")
           (unit 1)))))
@@
     (instances
       (project "pen_research"
-        (path "/8dc8c6c6-b52c-4ea1-b54e-983058d7675b/f0a18f19-96a9-433d-b9f0-5a690030b810"
+        (path "/f9a5e985-59a4-50af-9b9a-f23ea55006e2/ddb8b498-860e-5487-980d-a3b64ae1ae94"
           (reference "C65")
           (unit 1)))))
@@
       (justify left bottom))
 )
-  (text "IN/IN drive: PWM on one input, other low = drive/brake (slow decay); both low + SLEEP low = coast. Centre-aligned PWM, current sampled at period centre."
+  (text "IN/IN drive (DRV8212P truth table, VERIFY): slow decay = one input held high, the other driven with the inverted duty, i.e. drive (1,0) / brake (1,1). PWM on one input with the other low is drive/coast (fast decay). nSLEEP low = sleep, outputs Hi-Z. Centre-aligned PWM, current sampled at period centre."
     (exclude_from_sim no)
     (at 20 255.00 0)
